File: kicad/lm317 v3.1/lm317.kicad_pcb (KiCad board)
At the start: 2 copper layers, 28 x 31.5 mm, 9 parts, among them J1 VIN, J2 VOUT, U1 LM317

Commit message: fixed LM317 silk screen issue - cleaned up structure
Other:
- board text added: "LM317 - rev 3.1 shaunclarke.co.uk"
- board text removed: "LM317 - rev 3.0 shaunclarke.co.uk"
Changed lines of the file:
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@@
 			(outputformat 1)
 			(mirror no)
-			(drillshape 1)
+			(drillshape 0)
 			(scaleselection 1)
-			(outputdirectory "")
+			(outputdirectory "../../gerber/out")
 		)
 	)
@@
 		(property "Value" "VIN"
 			(at 0 4.92 0)
-			(layer "F.Fab")
+			(layer "F.SilkS")
 			(effects
 				(font
@@
 		)
 	)
-	(gr_text "LM317 - rev 3.0\nshaunclarke.co.uk"
+	(gr_text "LM317 - rev 3.1\nshaunclarke.co.uk"
 		(at 130.5 116 90)
 		(layer "F.SilkS")
